Commit message: feat: Intégration complète Gazebo (Inerties, Frictions, Caméra Plugin) dans l'URDF

File: urdf/robot_core.xacro (robot description, xacro)
@@ -6,9 +6,4 @@
     <material name="black"><color rgba="0 0 0 1"/></material>
     <link name="base_link"></link>
-    <joint name="base_footprint_joint" type="fixed">
-        <parent link="base_link"/><child link="base_footprint"/>
-        <origin xyz="0 0 0" rpy="0 0 0"/>
-    </joint>
-    <link name="base_footprint"></link>
     <joint name="chassis_joint" type="fixed">
         <parent link="base_link"/><child link="chassis"/>
@@ -18,26 +13,47 @@
         <visual>
             <origin xyz="0.15 0 0.075"/><geometry><box size="0.3 0.3 0.15"/></geometry>
-            <material name="white"/>
+            <material name="orange"/>
         </visual>
         <collision>
             <origin xyz="0.15 0 0.075"/><geometry><box size="0.3 0.3 0.15"/></geometry>
         </collision>
+        <inertial>
+            <origin xyz="0.15 0 0.075" rpy="0 0 0"/>
+            <mass value="0.5"/>
+            <inertia ixx="0.0046" ixy="0.0" ixz="0.0" iyy="0.0046" iyz="0.0" izz="0.0075"/>
+        </inertial>
     </link>
+    <gazebo reference="chassis">
+        <material>Gazebo/Orange</material>
+    </gazebo>
     <joint name="left_wheel_joint" type="continuous">
         <parent link="base_link"/><child link="left_wheel"/>
-        <origin xyz="0 0.175 0" rpy="-1.57 0 0"/><axis xyz="0 0 1"/>
+        <origin xyz="0 0.175 0" rpy="-1.5708 0 0"/><axis xyz="0 0 1"/>
     </joint>
     <link name="left_wheel">
         <visual><geometry><cylinder radius="0.05" length="0.04"/></geometry><material name="blue"/></visual>
         <collision><geometry><cylinder radius="0.05" length="0.04"/></geometry></collision>
+        <inertial>
+            <mass value="0.1"/><inertia ixx="7.5e-5" ixy="0" ixz="0" iyy="7.5e-5" iyz="0" izz="1.25e-4"/>
+        </inertial>
     </link>
+    <gazebo reference="left_wheel">
+        <material>Gazebo/Blue</material>
+        <mu1 value="0.2"/><mu2 value="0.2"/> </gazebo>
     <joint name="right_wheel_joint" type="continuous">
         <parent link="base_link"/><child link="right_wheel"/>
-        <origin xyz="0 -0.175 0" rpy="1.57 0 0"/><axis xyz="0 0 -1"/>
+        <origin xyz="0 -0.175 0" rpy="1.5708 0 0"/><axis xyz="0 0 -1"/>
     </joint>
     <link name="right_wheel">
         <visual><geometry><cylinder radius="0.05" length="0.04"/></geometry><material name="blue"/></visual>
         <collision><geometry><cylinder radius="0.05" length="0.04"/></geometry></collision>
+        <inertial>
+            <mass value="0.1"/><inertia ixx="7.5e-5" ixy="0" ixz="0" iyy="7.5e-5" iyz="0" izz="1.25e-4"/>
+        </inertial>
     </link>
+    <gazebo reference="right_wheel">
+        <material>Gazebo/Blue</material>
+        <mu1 value="0.2"/><mu2 value="0.2"/>
+    </gazebo>
     <joint name="caster_wheel_joint" type="fixed">
         <parent link="chassis"/><child link="caster_wheel"/>
@@ -47,4 +63,10 @@
         <visual><geometry><sphere radius="0.05"/></geometry><material name="black"/></visual>
         <collision><geometry><sphere radius="0.05"/></geometry></collision>
+        <inertial>
+            <mass value="0.1"/><inertia ixx="1e-4" ixy="0" ixz="0" iyy="1e-4" iyz="0" izz="1e-4"/>
+        </inertial>
     </link>
+    <gazebo reference="caster_wheel">
+        <material>Gazebo/Black</material>
+        <mu1 value="0.001"/><mu2 value="0.001"/> </gazebo>
 </robot>
